Commit message: Phase 6: Nav2 navigation, safety gateway and RViz configuration
AMCL + NavFn + Regulated Pure Pursuit + collision monitor + keepout filter. Fixes found
by measurement: outline-only map (AMCL wall bias), shrunk stop polygon (undocking stall),
narrowed lidar FOV and flush bumpers (phantom obstacles), server timeouts.

Co-Authored-By: Claude Opus 5.5 <noreply@anthropic.com>
Claude-Session: https://claude.ai/code/session_01J4fmJdpgG6N7SCchzQG4hL

File: ros2_ws/src/uco_description/urdf/agv.urdf.xacro (robot description, xacro)
@@ -25,4 +25,8 @@
   <xacro:property name="wheel_mass" value="5.0"/>
   <xacro:property name="lidar_z" value="0.20"/>   <!-- scan plane height above ground -->
+  <!-- Half field of view: 132 deg, not 135. At exactly 135 deg the edge ray runs parallel to the
+       chassis face 4.5 cm away and returned spurious ranges (phantom obstacles). The two corner
+       scanners still overlap to 360 deg: front covers -87..177 deg, rear 93..357 deg. -->
+  <xacro:property name="lidar_half_fov" value="${radians(132)}"/>
   <xacro:macro name="box_inertia" params="m x y z">
     <inertial><mass value="${m}"/>
@@ -45,10 +49,10 @@
     </visual>
     <visual name="bumper_front">
-      <origin xyz="${L/2 - 0.02} 0 ${chassis_bottom + 0.06 - wheel_r}"/>
+      <origin xyz="${L/2 - 0.025} 0 ${chassis_bottom + 0.06 - wheel_r}"/>  <!-- flush, no self-hits -->
       <geometry><box size="0.05 ${W - 0.1} 0.08"/></geometry>
       <material name="yellow"/>
     </visual>
     <visual name="bumper_rear">
-      <origin xyz="${-L/2 + 0.02} 0 ${chassis_bottom + 0.06 - wheel_r}"/>
+      <origin xyz="${-L/2 + 0.025} 0 ${chassis_bottom + 0.06 - wheel_r}"/>
       <geometry><box size="0.05 ${W - 0.1} 0.08"/></geometry>
       <material name="yellow"/>
@@ -144,6 +148,5 @@
   <xacro:caster name="rear" x="${-caster_x}"/>
   <!-- ===================== sensors ===================== -->
-  <!-- 270 deg safety lidar mounted just outside a chassis corner, facing diagonally outwards.
-       Its +-135 deg field of view then grazes the two adjacent chassis faces without hitting them. -->
+  <!-- Safety lidar mounted just outside a chassis corner, facing diagonally outwards. -->
   <xacro:macro name="corner_lidar" params="name x y yaw topic">
     <link name="${name}_link">
@@ -168,8 +171,8 @@
           <scan>
             <horizontal>
-              <samples>271</samples>
+              <samples>265</samples>
               <resolution>1</resolution>
-              <min_angle>${-3*pi/4}</min_angle>
-              <max_angle>${3*pi/4}</max_angle>
+              <min_angle>${-lidar_half_fov}</min_angle>
+              <max_angle>${lidar_half_fov}</max_angle>
             </horizontal>
             <vertical><samples>1</samples><min_angle>0</min_angle><max_angle>0</max_angle></vertical>
