Commit message: Phases 12-14: safety supervisor, fault injection, scenario runner, dashboard, metrics
Safety core with watchdogs, zones and e-stop gate; fault injector with 9 fault types;
scenario runner with fault_suite (38/38 checks passed in Gazebo); web dashboard; metrics
recorder and plotting. Performance: C++ /clock throttle and single-threaded rclpy
executors bring the full stack from RTF 0.1-0.3 to ~1.0. 114 tests pass.

Co-Authored-By: Claude Opus 5.5 <noreply@anthropic.com>
Claude-Session: https://claude.ai/code/session_01J4fmJdpgG6N7SCchzQG4hL

File: ros2_ws/src/uco_description/urdf/agv.urdf.xacro (robot description, xacro)
@@ -272,5 +272,5 @@
       <odom_topic>/${ns}/ground_truth</odom_topic>
       <tf_topic>/${ns}/ground_truth_tf</tf_topic>
-      <odom_publish_frequency>20</odom_publish_frequency>
+      <odom_publish_frequency>10</odom_publish_frequency>
       <dimensions>2</dimensions>
     </plugin>
